Commit message: Update humanoid_robot.urdf.xacro

File: urdf/humanoid_robot.urdf.xacro (robot description, xacro)
@@ -5,7 +5,11 @@
   <xacro:property name="PI" value="3.1415926535897931"/>
   <gazebo>
-  <plugin name="gazebo_ros_control" filename="libgazebo_ros_control.so">
-    <robotNamespace>/humanoid</robotNamespace>
-  </plugin>
+    <plugin name="gazebo_ros_control" filename="libgazebo_ros_control.so">
+      <robotNamespace>/humanoid</robotNamespace>
+    </plugin>
+  </gazebo>
+  <!-- Ensure robot spawns upright -->
+  <gazebo reference="base_link">
+    <pose>0 0 0.9 0 0 0</pose>
   </gazebo>
   <!-- Material definitions -->
@@ -152,5 +156,5 @@
       <material name="blue"/>
     </visual>
-    <collision>
+    <collision name="foot_left_collision">
       <geometry>
         <box size="0.24 0.12 0.04"/>
@@ -277,5 +281,5 @@
       <material name="blue"/>
     </visual>
-    <collision>
+    <collision name="foot_right_collision">
       <geometry>
         <box size="0.24 0.12 0.04"/>
@@ -332,12 +336,12 @@
     </sensor>
   </gazebo>
-  <!-- Transmissions for joints with position controllers -->
+  <!-- Transmissions for joints with effort controllers -->
   <transmission name="knee_left_trans">
     <type>transmission_interface/SimpleTransmission</type>
     <joint name="knee_left">
-      <hardwareInterface>hardware_interface/PositionJointInterface</hardwareInterface>
+      <hardwareInterface>hardware_interface/EffortJointInterface</hardwareInterface>
     </joint>
     <actuator name="knee_left_motor">
-      <hardwareInterface>hardware_interface/PositionJointInterface</hardwareInterface>
+      <hardwareInterface>hardware_interface/EffortJointInterface</hardwareInterface>
       <mechanicalReduction>1</mechanicalReduction>
     </actuator>
@@ -346,8 +350,8 @@
     <type>transmission_interface/SimpleTransmission</type>
     <joint name="knee_right">
-      <hardwareInterface>hardware_interface/PositionJointInterface</hardwareInterface>
+      <hardwareInterface>hardware_interface/EffortJointInterface</hardwareInterface>
     </joint>
     <actuator name="knee_right_motor">
-      <hardwareInterface>hardware_interface/PositionJointInterface</hardwareInterface>
+      <hardwareInterface>hardware_interface/EffortJointInterface</hardwareInterface>
       <mechanicalReduction>1</mechanicalReduction>
     </actuator>
@@ -356,8 +360,8 @@
     <type>transmission_interface/SimpleTransmission</type>
     <joint name="hip_pitch_left">
-      <hardwareInterface>hardware_interface/PositionJointInterface</hardwareInterface>
+      <hardwareInterface>hardware_interface/EffortJointInterface</hardwareInterface>
     </joint>
     <actuator name="hip_pitch_left_motor">
-      <hardwareInterface>hardware_interface/PositionJointInterface</hardwareInterface>
+      <hardwareInterface>hardware_interface/EffortJointInterface</hardwareInterface>
       <mechanicalReduction>1</mechanicalReduction>
     </actuator>
@@ -366,8 +370,8 @@
     <type>transmission_interface/SimpleTransmission</type>
     <joint name="hip_pitch_right">
-      <hardwareInterface>hardware_interface/PositionJointInterface</hardwareInterface>
+      <hardwareInterface>hardware_interface/EffortJointInterface</hardwareInterface>
     </joint>
     <actuator name="hip_pitch_right_motor">
-      <hardwareInterface>hardware_interface/PositionJointInterface</hardwareInterface>
+      <hardwareInterface>hardware_interface/EffortJointInterface</hardwareInterface>
       <mechanicalReduction>1</mechanicalReduction>
     </actuator>
@@ -376,8 +380,8 @@
     <type>transmission_interface/SimpleTransmission</type>
     <joint name="hip_roll_left">
-      <hardwareInterface>hardware_interface/PositionJointInterface</hardwareInterface>
+      <hardwareInterface>hardware_interface/EffortJointInterface</hardwareInterface>
     </joint>
     <actuator name="hip_roll_left_motor">
-      <hardwareInterface>hardware_interface/PositionJointInterface</hardwareInterface>
+      <hardwareInterface>hardware_interface/EffortJointInterface</hardwareInterface>
       <mechanicalReduction>1</mechanicalReduction>
     </actuator>
@@ -386,12 +390,12 @@
     <type>transmission_interface/SimpleTransmission</type>
     <joint name="hip_roll_right">
-      <hardwareInterface>hardware_interface/PositionJointInterface</hardwareInterface>
+      <hardwareInterface>hardware_interface/EffortJointInterface</hardwareInterface>
     </joint>
     <actuator name="hip_roll_right_motor">
-      <hardwareInterface>hardware_interface/PositionJointInterface</hardwareInterface>
-      <mechanicalReduction>1</mechanicalReduction>
-    </actuator>
-  </transmission>
-  <!-- Ankle joints remain effort-based for LQR balance -->
+      <hardwareInterface>hardware_interface/EffortJointInterface</hardwareInterface>
+      <mechanicalReduction>1</mechanicalReduction>
+    </actuator>
+  </transmission>
+  <!-- Ankle joints remain effort-based -->
   <transmission name="ankle_pitch_left_trans">
     <type>transmission_interface/SimpleTransmission</type>
